Commit message: Update 2023.04.18 12:51

File: robots/cyberdog_description/urdf/cyberdog_description.urdf (robot description, URDF)
Before this commit: robot cyberdog_description, 19 links, 18 joints
Links:
- link FL_foot: mass 0.06 -> 0.00
- link FR_foot: mass 0.06 -> 0.00
- link RR_foot: mass 0.06 -> 0.00

Commit message: change feet mass

File: robots/cyberdog_description/urdf/cyberdog_description.urdf (robot description, URDF)
Before this commit: robot cyberdog_description, 19 links, 18 joints
Links:
- link FL_foot: mass 0.00 -> 0.06
- link FR_foot: mass 0.00 -> 0.06
- link RR_foot: mass 0.00 -> 0.06

Commit message: change feet mass to 0.026

File: robots/cyberdog_description/urdf/cyberdog_description.urdf (robot description, URDF)
Before this commit: robot cyberdog_description, 19 links, 18 joints
Links:
- link FL_foot: mass 0.06 -> 0.026
- link FR_foot: mass 0.06 -> 0.026
- link RL_foot: mass 0.06 -> 0.026
- link RR_foot: mass 0.06 -> 0.026

Commit message: add yaml

File: robots/cyberdog_description/urdf/cyberdog_description.urdf (robot description, URDF)
Before this commit: robot cyberdog_description, 19 links, 18 joints
Joints:
- joint FL_calf_joint: limit lower=-2.478 upper=-0.506 effort=24 velocity=12 -> lower=-2.478 upper=-0.506 effort=240 velocity=12
- joint FL_hip_joint: limit lower=-0.75 upper=0.75 effort=17 velocity=12 -> lower=-0.75 upper=0.75 effort=170 velocity=12
- joint FL_thigh_joint: limit lower=-1.257 upper=4.363 effort=24 velocity=12 -> lower=-1.257 upper=4.363 effort=240 velocity=12
- joint FR_calf_joint: limit lower=-2.478 upper=-0.506 effort=24 velocity=12 -> lower=-2.478 upper=-0.506 effort=240 velocity=12
- joint FR_hip_joint: limit lower=-0.75 upper=0.75 effort=17 velocity=12 -> lower=-0.75 upper=0.75 effort=170 velocity=12
- joint FR_thigh_joint: limit lower=-1.257 upper=4.363 effort=24 velocity=12 -> lower=-1.257 upper=4.363 effort=240 velocity=12
- joint RL_calf_joint: limit lower=-2.478 upper=-0.506 effort=24 velocity=12 -> lower=-2.478 upper=-0.506 effort=240 velocity=12
- joint RL_hip_joint: limit lower=-0.75 upper=0.75 effort=17 velocity=12 -> lower=-0.75 upper=0.75 effort=170 velocity=12
- joint RL_thigh_joint: limit lower=-2.01 upper=3.49 effort=24 velocity=12 -> lower=-2.01 upper=3.49 effort=240 velocity=12
- joint RR_calf_joint: limit lower=-2.478 upper=-0.506 effort=24 velocity=12 -> lower=-2.478 upper=-0.506 effort=240 velocity=12
- joint RR_hip_joint: limit lower=-0.75 upper=0.75 effort=17 velocity=12 -> lower=-0.75 upper=0.75 effort=170 velocity=12
- joint RR_thigh_joint: limit lower=-2.01 upper=3.49 effort=24 velocity=12 -> lower=-2.01 upper=3.49 effort=240 velocity=12
